File: SolarTelescope_LED/SolarTelescope_LED_PCB/SolarTelescope_LED_PCB.kicad_pcb (KiCad board)
At the start: 2 copper layers, 152.4 x 63.5 mm, 49 parts, among them J1 Screw_Terminal_01x05, U1 LM324, U2 LM324, U3 LM324

Commit message: Version B.
Parts:
- removed the G*** at (114.9, 98.4)
- removed J1: Screw_Terminal_01x05, TerminalBlock_Phoenix:TerminalBlock_Phoenix_MKDS-3-5-5.08_1x05_P5.08mm_Horizontal
- added J2: Screw_Terminal_01x06, TerminalBlock_Phoenix:TerminalBlock_Phoenix_MKDS-1,5-6_1x06_P5.00mm_Horizontal, B.Cu at (75.6, 100.6)
- moved R4 11.7 mm to (114.9, 90.2)
- moved R3 11.6 mm to (114.9, 101.3)
- moved U1 11.2 mm to (101.6, 88.7)
- moved R2 6.48 mm to (91.4, 98.4)
- moved R1 6.31 mm to (91.4, 93.0)
- moved C1 6.02 mm to (87.0, 108.6), turned to 90 degrees
- moved R14 5.78 mm to (91.4, 87.3)
Connections:
- C1 pad 1: +15VDC -> +Vcc
- C1 pad 2: GND -> -Vcc
- R1 pad 1: +15VDC -> Vtop
- R13 pad 2: GND -> Vbottom
- U1 pad 11: GND -> -Vcc
- U1 pad 4: +15VDC -> +Vcc
- U2 pad 11: GND -> -Vcc
- U2 pad 4: +15VDC -> +Vcc
- U3 pad 11: GND -> -Vcc
- U3 pad 4: +15VDC -> +Vcc
Routing:
- net +15VDC: track 143.2 -> 0.00 mm
- net GND: track 390.9 -> 255.3 mm, vias 1 -> 0
- net -Vcc: track 0.00 -> 132.2 mm
- net Vbottom: track 0.00 -> 125.5 mm, vias 0 -> 1
- net +Vcc: track 0.00 -> 122.2 mm
- net Vtop: track 0.00 -> 18.5 mm
- net Net-(U1D--): track 31.1 -> 20.2 mm
- net Net-(U1B--): track 23.9 -> 30.6 mm
- net Net-(R17-Pad1): track 19.2 -> 13.0 mm
- net Net-(R14-Pad1): track 4.76 -> 10.4 mm
- net Net-(R15-Pad1): track 30.0 -> 34.5 mm
- net Net-(U1A--): track 11.0 -> 14.7 mm
- net Vin: track 150.8 -> 147.3 mm
- net Net-(D1-A): track 23.0 -> 24.9 mm
- net Net-(U1C--): track 13.6 -> 15.3 mm
Other:
- board text added: "+Vcc"
- board text added: "-Vcc"
- board text added: "Vb"
- board text added: "Vt"
- board text removed: "V1"
- board text removed: "V2"
