File: SolarTelescope_LED/SolarTelescope_LED_PCB/SolarTelescope_LED_PCB.kicad_sch (KiCad schematic)
At the start: 42 parts, among them J1 Screw_Terminal_01x05, U1 LM324, U2 LM324, U3 LM324

Commit message: Version B.
Parts:
- removed J1: Screw_Terminal_01x05, TerminalBlock_Phoenix:TerminalBlock_Phoenix_MKDS-3-5-5.08_1x05_P5.08mm_Horizontal, symbol Connector:Screw_Terminal_01x05
- added J2: Screw_Terminal_01x06, TerminalBlock_Phoenix:TerminalBlock_Phoenix_MKDS-1,5-6_1x06_P5.00mm_Horizontal, symbol Connector:Screw_Terminal_01x06
- R1: value 48k -> 16.9k
- R10, R11, R12, R2, R3, R4, R5, R6, R7, R8, R9: value 1k -> 750
- R13: value 1k -> 49.9k
Connections:
- net GND: now also J2.6 (Pin_6); no longer C1.2, R13.2, U1.11 (V-), U2.11 (V-), U3.11 (V-)
- net Vin: now also J2.1 (Pin_1)
- net +15VDC renamed +Vcc
- net +Vcc: now also J2.2 (Pin_2); no longer R1.1
- new net -Vcc: C1.2, J2.3 (Pin_3), U1.11 (V-), U2.11 (V-), U3.11 (V-)
- new net Vbottom: J2.5 (Pin_5), R13.2
- new net Vtop: J2.4 (Pin_4), R1.1
